File: kicad/Circuito de Comando.kicad_pcb (KiCad board)
At the start: 2 copper layers, 68 parts, among them J1 sg3525, J2 Alimentação, J3 Vs, J4 Potência, J5 Carga, J6 Carga-2, J7 PID, J8 Conversor CC, J9 Jumper PID, Q1 BC337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

Commit message: add report
Parts:
- removed the C1 at (41.5, 41.6)
- removed the C2 at (67.8, 33.3)
- removed the D1 at (71.8, 36.8)
- removed the D2 at (71.8, 44.6)
- removed the D3 at (100.1, 44.5)
- removed the D4 at (113.0, 50.2)
- removed the J1 at (52.1, 31.8)
- removed the J2 at (91.3, 31.5)
- removed the J7 at (76.0, 31.5)
- removed the J8 at (101.7, 31.5)
- removed the J9 at (43.2, 35.8)
- removed the Q1 at (77.5, 55.9)
- removed the Q2 at (105.4, 55.9)
- removed the Q3 at (91.2, 55.9)
- removed the Q4 at (125.7, 35.6)
- removed the R1 at (52.1, 27.1)
- removed the R3 at (76.5, 40.1)
- removed the R4 at (80.3, 40.1)
- removed the R5 at (84.1, 40.1)
- removed the R6 at (87.9, 40.1)
- removed the R7 at (110.5, 44.5)
- removed the R8 at (117.5, 50.2)
- removed the R9 at (47.0, 48.3)
- removed the RV1 at (39.4, 55.8)
- removed the RV2 at (44.6, 25.7)
Routing:
- net GND: track 612.1 -> 323.4 mm
- net VCC: track 190.5 -> 95.2 mm
- net Net-(J1-Pad2): track 160.8 -> 80.4 mm
- net Net-(Q2-Pad2): track 92.4 -> 46.2 mm
- net Net-(D3-Pad2): track 86.8 -> 43.4 mm
- net Net-(J8-Pad2): track 76.4 -> 38.2 mm
- net Net-(D4-Pad1): track 60.2 -> 30.1 mm
- net Net-(C1-Pad1): track 59.0 -> 29.5 mm
- net Net-(Q1-Pad1): track 52.8 -> 26.4 mm
- net Net-(J1-Pad1): track 45.3 -> 22.7 mm
- net Net-(D3-Pad1): track 38.5 -> 19.2 mm
- net Net-(J9-Pad2): track 34.5 -> 17.3 mm
- net Net-(D1-Pad1): track 27.6 -> 13.8 mm
- net Net-(J1-Pad6): track 16.3 -> 8.16 mm
- net Net-(Q1-Pad2): track 15.6 -> 7.80 mm
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