File: kicad/Circuito de Comando.sch (KiCad schematic (older format))
At the start: 43 parts, among them J1 sg3525, J2 Alimentação, J3 Vs, J4 Potência, J5 Carga, J6 Carga-2, J7 PID, J8 Conversor CC, J9 Jumper PID, Q1 BC337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

Commit message: add report
Parts:
- C2: value C -> 10nF
- R1: value R -> 10k
- RV1, RV2: value POT -> 50k
Changed lines of the file:
@@
 encoding utf-8
 Sheet 1 1
-Title "Projeto de Eletrônica de Potência"
+Title "Conversor Boost - Projeto de Eletrônica de Potência"
 Date "2018-05-30"
 Rev ""
@@
 P 2850 2250
 F 0 "R1" V 2750 2250 50  0000 C CNN
-F 1 "R" V 2850 2250 50  0000 C CNN
+F 1 "10k" V 2850 2250 50  0000 C CNN
 F 2 "Potentiometers:Potentiometer_WirePads" V 2780 2250 50  0001 C CNN
 F 3 "" H 2850 2250 50  0001 C CNN
@@
 P 2000 3400
 F 0 "RV1" H 1850 3450 50  0000 C CNN
-F 1 "POT" H 1850 3350 50  0000 C CNN
+F 1 "50k" H 1850 3350 50  0000 C CNN
 F 2 "Potentiometers:Potentiometer_Trimmer_ACP_CA6v_Horizontal" H 2000 3400 50  0001 C CNN
 F 3 "" H 2000 3400 50  0001 C CNN
@@
 P 1250 3500
 F 0 "RV2" V 1075 3500 50  0000 C CNN
-F 1 "POT" V 1150 3500 50  0000 C CNN
+F 1 "50k" V 1150 3500 50  0000 C CNN
 F 2 "Potentiometers:Potentiometer_Trimmer_ACP_CA6v_Horizontal" H 1250 3500 50  0001 C CNN
 F 3 "" H 1250 3500 50  0001 C CNN
@@
 P 3600 2500
 F 0 "C2" V 3750 2500 50  0000 L CNN
-F 1 "C" V 3850 2550 50  0000 L CNN
+F 1 "10nF" V 3850 2550 50  0000 L CNN
 F 2 "Capacitors_THT:CP_Radial_D8.0mm_P5.00mm" H 3638 2350 50  0001 C CNN
 F 3 "" H 3600 2500 50  0001 C CNN
